Commit message: problem statement 1 finished

File: src/two_scara_collaboration/urdf/scara_left.urdf.xacro (robot description, xacro)
@@ -56,13 +56,13 @@
   <link name="scara_left_link_1">
     <collision>
-      <origin xyz="0 0.5 0.05" rpy="0 0 0"/>
-      <geometry>
-        <box size="0.1 1.1 0.1"/>
-      </geometry>
-    </collision>
-    <visual>
-      <origin xyz="0 0.5 0.05" rpy="0 0 0"/>
-      <geometry>
-        <box size="0.1 1.1 0.1"/>
+      <origin xyz="0 0.75 0.05" rpy="0 0 0"/>
+      <geometry>
+        <box size="0.1 1.6 0.1"/>
+      </geometry>
+    </collision>
+    <visual>
+      <origin xyz="0 0.75 0.05" rpy="0 0 0"/>
+      <geometry>
+        <box size="0.1 1.6 0.1"/>
       </geometry>
       <material name="blue">
@@ -83,5 +83,5 @@
     <parent link="scara_left_link_1"/>
     <child link="scara_left_link_2"/>
-    <origin xyz="0 1 0.1" rpy="0 0 0"/>
+    <origin xyz="0 1.5 0.1" rpy="0 0 0"/> <!-- L1 Increased to 1.5 -->
     <axis xyz="0 0 1"/>
     <limit effort="100" velocity="100" lower="-3.00" upper="3.00"/>
@@ -89,13 +89,13 @@
   <link name="scara_left_link_2">
     <collision>
-      <origin xyz="0 0.4 0.05" rpy="0 0 0"/>
-      <geometry>
-        <box size="0.1 0.9 0.1"/>
-      </geometry>
-    </collision>
-    <visual>
-      <origin xyz="0 0.4 0.05" rpy="0 0 0"/>
-      <geometry>
-        <box size="0.1 0.9 0.1"/>
+      <origin xyz="0 0.5 0.05" rpy="0 0 0"/>
+      <geometry>
+        <box size="0.1 1.1 0.1"/>
+      </geometry>
+    </collision>
+    <visual>
+      <origin xyz="0 0.5 0.05" rpy="0 0 0"/>
+      <geometry>
+        <box size="0.1 1.1 0.1"/>
       </geometry>
       <material name="cyan">
@@ -116,7 +116,7 @@
     <parent link="scara_left_link_2"/>
     <child link="scara_left_gripper_base_link"/>
-    <origin xyz="0 0.8 0" rpy="0 0 0"/>
+    <origin xyz="0 1.0 0" rpy="0 0 0"/> <!-- L2 Increased to 1.0 -->
     <axis xyz="0 0 1"/>
-    <limit effort="100" velocity="100" lower="-0.05" upper="0.0"/>
+    <limit effort="100" velocity="100" lower="-0.6" upper="0.0"/>
   </joint>
   <link name="scara_left_gripper_base_link">

File: src/two_scara_collaboration/urdf/scara_right.urdf.xacro (robot description, xacro)
@@ -56,16 +56,16 @@
   <link name="scara_right_link_1">
     <collision>
-      <origin xyz="0 0.5 0.05" rpy="0 0 0"/>
-      <geometry>
-        <box size="0.1 1.1 0.1"/>
-      </geometry>
-    </collision>
-    <visual>
-      <origin xyz="0 0.5 0.05" rpy="0 0 0"/>
-      <geometry>
-        <box size="0.1 1.1 0.1"/>
-      </geometry>
-      <material name="red">
-        <color rgba="1 0 0 1"/>
+      <origin xyz="0 0.75 0.05" rpy="0 0 0"/>
+      <geometry>
+        <box size="0.1 1.6 0.1"/>
+      </geometry>
+    </collision>
+    <visual>
+      <origin xyz="0 0.75 0.05" rpy="0 0 0"/>
+      <geometry>
+        <box size="0.1 1.6 0.1"/>
+      </geometry>
+      <material name="blue">
+        <color rgba="0 0 1 1"/>
       </material>
     </visual>
@@ -77,5 +77,5 @@
   </link>
   <gazebo reference="scara_right_link_1">
-    <material>Gazebo/Red</material>
+    <material>Gazebo/Blue</material>
   </gazebo>
   <!-- Joint 2 (Rotation 2) -->
@@ -83,5 +83,5 @@
     <parent link="scara_right_link_1"/>
     <child link="scara_right_link_2"/>
-    <origin xyz="0 1 0.1" rpy="0 0 0"/>
+    <origin xyz="0 1.5 0.1" rpy="0 0 0"/> <!-- L1 Increased to 1.5 -->
     <axis xyz="0 0 1"/>
     <limit effort="100" velocity="100" lower="-3.00" upper="3.00"/>
@@ -89,16 +89,16 @@
   <link name="scara_right_link_2">
     <collision>
-      <origin xyz="0 0.4 0.05" rpy="0 0 0"/>
-      <geometry>
-        <box size="0.1 0.9 0.1"/>
-      </geometry>
-    </collision>
-    <visual>
-      <origin xyz="0 0.4 0.05" rpy="0 0 0"/>
-      <geometry>
-        <box size="0.1 0.9 0.1"/>
-      </geometry>
-      <material name="green">
-        <color rgba="0 1 0 1"/>
+      <origin xyz="0 0.5 0.05" rpy="0 0 0"/>
+      <geometry>
+        <box size="0.1 1.1 0.1"/>
+      </geometry>
+    </collision>
+    <visual>
+      <origin xyz="0 0.5 0.05" rpy="0 0 0"/>
+      <geometry>
+        <box size="0.1 1.1 0.1"/>
+      </geometry>
+      <material name="cyan">
+        <color rgba="0 1 1 1"/>
       </material>
     </visual>
@@ -110,5 +110,5 @@
   </link>
   <gazebo reference="scara_right_link_2">
-    <material>Gazebo/Green</material>
+    <material>Gazebo/SkyBlue</material>
   </gazebo>
   <!-- Gripper Base Joint -->
@@ -116,7 +116,7 @@
     <parent link="scara_right_link_2"/>
     <child link="scara_right_gripper_base_link"/>
-    <origin xyz="0 0.8 0" rpy="0 0 0"/>
+    <origin xyz="0 1.0 0" rpy="0 0 0"/> <!-- L2 Increased to 1.0 -->
     <axis xyz="0 0 1"/>
-    <limit effort="100" velocity="100" lower="-0.05" upper="0.0"/>
+    <limit effort="100" velocity="100" lower="-0.6" upper="0.0"/>
   </joint>
   <link name="scara_right_gripper_base_link">

File: src/two_scara_collaboration/urdf/world.urdf.xacro (robot description, xacro)
@@ -15,5 +15,5 @@
     <parent link="world"/>
     <child link="scara_left_base_link"/>
-    <origin xyz="2 -1 0.2" rpy="0 0 0"/>
+    <origin xyz="2 -2 0.2" rpy="0 0 0"/>
   </joint>
   <xacro:scara_left_robot/>
@@ -25,4 +25,32 @@
   </joint>
   <xacro:scara_right_robot/>
+  <!-- Basket -->
+  <joint name="basket_joint" type="fixed">
+    <parent link="world"/>
+    <child link="basket_link"/>
+    <origin xyz="2.0 -4.0 0.1" rpy="0 0 0"/>
+  </joint>
+  <link name="basket_link">
+    <visual>
+      <geometry>
+        <box size="0.5 0.5 0.2"/>
+      </geometry>
+      <material name="red">
+        <color rgba="1 0 0 1"/>
+      </material>
+    </visual>
+    <collision>
+      <geometry>
+        <box size="0.5 0.5 0.2"/>
+      </geometry>
+    </collision>
+    <inertial>
+      <mass value="10"/>
+      <inertia ixx="0.1" ixy="0" ixz="0" iyy="0.1" iyz="0" izz="0.1"/>
+    </inertial>
+  </link>
+  <gazebo reference="basket_link">
+    <material>Gazebo/Red</material>
+  </gazebo>
   <!-- Global ros2_control plugin -->
   <gazebo>

Commit message: feat: Implement two SCARA robot collaboration in ROS2 with Gazebo simulation, kinematics, and control.

File: src/two_scara_collaboration/urdf/scara_left.urdf.xacro (robot description, xacro)
@@ -1,4 +1,4 @@
 <robot xmlns:xacro="http://www.ros.org/wiki/xacro" name="scara_left">
-<xacro:macro name="scara_left_robot">
+<xacro:macro name="scara_left_robot" params="thickness:=0.1">
   <!-- ROS2 Control -->
   <ros2_control name="LeftGazeboSystem" type="system">
@@ -28,5 +28,5 @@
       <origin xyz="0 0 0.2" rpy="0 0 0"/>
       <geometry>
-        <cylinder length="0.4" radius="0.1"/>
+        <cylinder length="0.4" radius="${thickness}"/>
       </geometry>
     </collision>
@@ -34,5 +34,5 @@
       <origin xyz="0 0 0.2" rpy="0 0 0"/>
       <geometry>
-        <cylinder length="0.4" radius="0.1"/>
+        <cylinder length="0.4" radius="${thickness}"/>
       </geometry>
       <material name="gray">
@@ -56,13 +56,13 @@
   <link name="scara_left_link_1">
     <collision>
-      <origin xyz="0 0.75 0.05" rpy="0 0 0"/>
-      <geometry>
-        <box size="0.1 1.6 0.1"/>
-      </geometry>
-    </collision>
-    <visual>
-      <origin xyz="0 0.75 0.05" rpy="0 0 0"/>
-      <geometry>
-        <box size="0.1 1.6 0.1"/>
+      <origin xyz="0 0.75 ${thickness/2}" rpy="0 0 0"/>
+      <geometry>
+        <box size="${thickness} 1.6 ${thickness}"/>
+      </geometry>
+    </collision>
+    <visual>
+      <origin xyz="0 0.75 ${thickness/2}" rpy="0 0 0"/>
+      <geometry>
+        <box size="${thickness} 1.6 ${thickness}"/>
       </geometry>
       <material name="blue">
@@ -89,13 +89,13 @@
   <link name="scara_left_link_2">
     <collision>
-      <origin xyz="0 0.5 0.05" rpy="0 0 0"/>
-      <geometry>
-        <box size="0.1 1.1 0.1"/>
-      </geometry>
-    </collision>
-    <visual>
-      <origin xyz="0 0.5 0.05" rpy="0 0 0"/>
-      <geometry>
-        <box size="0.1 1.1 0.1"/>
+      <origin xyz="0 0.5 ${thickness/2}" rpy="0 0 0"/>
+      <geometry>
+        <box size="${thickness} 1.1 ${thickness}"/>
+      </geometry>
+    </collision>
+    <visual>
+      <origin xyz="0 0.5 ${thickness/2}" rpy="0 0 0"/>
+      <geometry>
+        <box size="${thickness} 1.1 ${thickness}"/>
       </geometry>
       <material name="cyan">

File: src/two_scara_collaboration/urdf/scara_right.urdf.xacro (robot description, xacro)
@@ -1,4 +1,4 @@
 <robot xmlns:xacro="http://www.ros.org/wiki/xacro" name="scara_right">
-<xacro:macro name="scara_right_robot">
+<xacro:macro name="scara_right_robot" params="thickness:=0.1">
   <!-- ROS2 Control -->
   <ros2_control name="RightGazeboSystem" type="system">
@@ -28,5 +28,5 @@
       <origin xyz="0 0 0.2" rpy="0 0 0"/>
       <geometry>
-        <cylinder length="0.4" radius="0.1"/>
+        <cylinder length="0.4" radius="${thickness}"/>
       </geometry>
     </collision>
@@ -34,5 +34,5 @@
       <origin xyz="0 0 0.2" rpy="0 0 0"/>
       <geometry>
-        <cylinder length="0.4" radius="0.1"/>
+        <cylinder length="0.4" radius="${thickness}"/>
       </geometry>
       <material name="gray">
@@ -56,13 +56,13 @@
   <link name="scara_right_link_1">
     <collision>
-      <origin xyz="0 0.75 0.05" rpy="0 0 0"/>
-      <geometry>
-        <box size="0.1 1.6 0.1"/>
-      </geometry>
-    </collision>
-    <visual>
-      <origin xyz="0 0.75 0.05" rpy="0 0 0"/>
-      <geometry>
-        <box size="0.1 1.6 0.1"/>
+      <origin xyz="0 0.75 ${thickness/2}" rpy="0 0 0"/>
+      <geometry>
+        <box size="${thickness} 1.6 ${thickness}"/>
+      </geometry>
+    </collision>
+    <visual>
+      <origin xyz="0 0.75 ${thickness/2}" rpy="0 0 0"/>
+      <geometry>
+        <box size="${thickness} 1.6 ${thickness}"/>
       </geometry>
       <material name="blue">
@@ -89,13 +89,13 @@
   <link name="scara_right_link_2">
     <collision>
-      <origin xyz="0 0.5 0.05" rpy="0 0 0"/>
-      <geometry>
-        <box size="0.1 1.1 0.1"/>
-      </geometry>
-    </collision>
-    <visual>
-      <origin xyz="0 0.5 0.05" rpy="0 0 0"/>
-      <geometry>
-        <box size="0.1 1.1 0.1"/>
+      <origin xyz="0 0.5 ${thickness/2}" rpy="0 0 0"/>
+      <geometry>
+        <box size="${thickness} 1.1 ${thickness}"/>
+      </geometry>
+    </collision>
+    <visual>
+      <origin xyz="0 0.5 ${thickness/2}" rpy="0 0 0"/>
+      <geometry>
+        <box size="${thickness} 1.1 ${thickness}"/>
       </geometry>
       <material name="cyan">

File: src/two_scara_collaboration/urdf/world.urdf.xacro (robot description, xacro)
@@ -6,4 +6,6 @@
   <xacro:include filename="$(find two_scara_collaboration)/urdf/scara_right.urdf.xacro"/>
   <!-- Instantiate Elements -->
+  <!-- Arguments -->
+  <xacro:arg name="robot_thickness" default="0.1"/>
   <!-- Left Robot -->
   <joint name="scara_left_to_world" type="fixed">
@@ -12,5 +14,5 @@
     <origin xyz="2 -2 0.2" rpy="0 0 0"/>
   </joint>
-  <xacro:scara_left_robot/>
+  <xacro:scara_left_robot thickness="$(arg robot_thickness)"/>
   <!-- Right Robot -->
   <joint name="scara_right_to_world" type="fixed">
@@ -19,5 +21,5 @@
     <origin xyz="2 2 0.2" rpy="0 0 0"/>
   </joint>
-  <xacro:scara_right_robot/>
+  <xacro:scara_right_robot thickness="$(arg robot_thickness)"/>
   <!-- Global ros2_control plugin -->
   <gazebo>
